File: hardware/kicad/atlas.kicad_pcb (KiCad board)
At the start: 4 copper layers, 38.4 x 82.2 mm, 120 parts, among them J1 U262-161N-4BVC11, J2 +LIPO, J3 -LIPO, J4 HC-FPC-05-09-24RLTAG, Q1 DMG1012UW, Q2 DMG1012UW, Q4 PMV32UP, Q5 DMG1012UW, Q6 AO3407A, Q7 SI1308EDL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

Commit message: wip
Parts:
- removed JP1: GPS_VBCKP, Jumper:SolderJumper-3_P1.3mm_Open_RoundedPad1.0x1.5mm_NumberLabels
- removed Q2: DMG1012UW, Package_TO_SOT_SMD:SOT-323_SC-70
- removed R14: 1M, Resistor_SMD:R_0402_1005Metric
- added TP1: DL_TXD0, TestPoint:TestPoint_Pad_D1.0mm, F.Cu at (119.9, 51.8)
- added TP2: DL_RXD0, TestPoint:TestPoint_Pad_D1.0mm, F.Cu at (119.9, 49.7)
- C42, C44: value 0.1uF -> 100n
- C43: value 4.7uF -> 4u7
- C45: value 10uF -> 10u
- R5: value 10K -> 1M; footprint Resistor_SMD:R_0402_1005Metric -> Resistor_SMD:R_0603_1608Metric
- TP7: value BOOT_MODE0 -> BOOT_MODE1
- U10: footprint atlas:XCVR_L86-M33 -> atlas:L86-M33
Connections:
- C42 pad 1: /GPS/GPS_VBCKP -> +BATT
- C43 pad 1: /GPS/GPS_VBCKP -> +BATT
- R15 pad 1: /GPS/GPS_FORCE_ON -> /GNSS/GNSS_FORCE_ON
- R5 pad 2: /Main Controller/MPP_STS_READ -> /Main Controller/BOOT_MODE1
- U1 pad 10: /GPS/GPS_FORCE_ON -> /GNSS/GNSS_TXD
- U1 pad 11: /Main Controller/MPP_STS_READ -> /GNSS/GNSS_RXD
- U1 pad 21: /GPS/GPS_RXD -> Net-(U1-U0TXD/GPIO16/FSPICS0)
- U1 pad 22: /GPS/GPS_TXD -> Net-(U1-U0RXD/GPIO17/FSPICS1)
- U1 pad 28: /Main Controller/PWM -> /GNSS/GNSS_FORCE_ON
- U10 pad 1: /GPS/GPS_RXD -> /GNSS/GNSS_RXD
- U10 pad 10: unconnected-(U10-~{RESET}-Pad10) -> /Main Controller/BOOT_MODE1
- U10 pad 2: /GPS/GPS_TXD -> /GNSS/GNSS_TXD
- U10 pad 5: /GPS/GPS_VBCKP -> +BATT
- U10 pad 7: /GPS/GPS_FORCE_ON -> /GNSS/GNSS_FORCE_ON
- U10 pad 9: unconnected-(U10-NC-Pad9) -> (no net)
- U4 pad 19: /Main Controller/MPP_STATUS -> unconnected-(U4-STATUS[2]-Pad19)
Routing:
- net /GPS/GPS_TXD: track 58.5 -> 0.00 mm, vias 2 -> 0
- net /GPS/GPS_RXD: track 55.0 -> 0.00 mm, vias 2 -> 0
- net /GPS/GPS_VBCKP: track 33.5 -> 0.00 mm
- net +BATT: track 81.7 -> 115.2 mm
- net unconnected-(U4-STATUS[2]-Pad19): track 0.00 -> 8.55 mm, vias 0 -> 2
- net /Main Controller/MPP_STATUS: track 8.55 -> 0.00 mm, vias 2 -> 0
- net Net-(U1-U0TXD/GPIO16/FSPICS0): track 0.00 -> 5.41 mm
- net Net-(U1-U0RXD/GPIO17/FSPICS1): track 0.00 -> 2.85 mm
- net /GPS/GPS_FORCE_ON: vias 3 -> 0
- net /GNSS/GNSS_FORCE_ON: vias 0 -> 3

Commit message: update pcb
Parts:
- removed R5: 1M, Resistor_SMD:R_0603_1608Metric
- R15: footprint Resistor_SMD:R_0603_1608Metric -> Resistor_SMD:R_0402_1005Metric
- moved R15 25.7 mm to (103.9, 108.6)
- moved G*** 24.6 mm to (125.7, 54.4), turned to -90 degrees
- moved TP9 17.1 mm to (126.5, 49.3)
- moved C42 7.06 mm to (117.7, 90.4), turned to 180 degrees
- moved C44 5.69 mm to (121.3, 90.4), turned to 0 degrees
- moved C43 4.46 mm to (117.7, 88.9), turned to 180 degrees
- moved C45 3.06 mm to (121.3, 88.9), turned to 0 degrees
- moved R29 0.48 mm to (111.7, 48.5)
Connections:
- U1 pad 10: /GNSS/GNSS_TXD -> /GNSS/GNSS_RXD
- U1 pad 11: /GNSS/GNSS_RXD -> /GNSS/GNSS_TXD
Routing:
- net /GNSS/GNSS_FORCE_ON: track 0.00 -> 88.6 mm, vias 3 -> 1
- net /GPS/GPS_FORCE_ON: track 87.8 -> 0.00 mm
- net /GNSS/GNSS_TXD: track 0.00 -> 74.4 mm, vias 0 -> 4
- net /GNSS/GNSS_RXD: track 0.00 -> 72.8 mm, vias 0 -> 4
- net /Main Controller/BOOT_MODE1: track 23.9 -> 95.8 mm, vias 2 -> 3
- net +BATT: track 115.2 -> 96.1 mm, vias 3 -> 4
- net /Main Controller/CHIP_EN: track 44.1 -> 26.4 mm
- net /Main Controller/MPP_STS_READ: track 15.0 -> 0.00 mm, vias 2 -> 0
- net +3V3: track 194.0 -> 179.0 mm
- net unconnected-(U4-STATUS[2]-Pad19): track 8.55 -> 0.00 mm, vias 2 -> 0
- net GND: track 24.0 -> 19.8 mm, vias 210 -> 280
Other:
- board text added: "Atlas"
- board text added: "REVISION 1"
- board text added: "Teapotlabs Atlas"
- board text removed: "Plantpal"
- board text removed: "REVISION 5"
- board text removed: "SOIL MOISTURE SENSING"
