File: hardware/kicad/battery.kicad_sch (KiCad schematic)
At the start: 5 parts, among them J2 +LIPO, J3 -LIPO, Q6 AO3407A

Commit message: update schematics info
Other:
- title: Battery -> Teapotlabs Atlas
Changed lines of the file:
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@@
 	(paper "A5")
 	(title_block
-		(title "Battery")
-		(date "2024-04-06")
-		(rev "5")
+		(title "Teapotlabs Atlas")
+		(date "2024-10-25")
+		(rev "1")
 		(company "Teapot Laboratories")
 	)
