File: hardware/kicad/display.kicad_sch (KiCad schematic)
At the start: 19 parts, among them J4 HC-FPC-05-09-24RLTAG, Q7 SI1308EDL

Commit message: update schematics info
Other:
- title: Display -> Teapotlabs Atlas
Changed lines of the file:
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@@
 	(paper "A5")
 	(title_block
-		(title "Display")
-		(date "2024-04-06")
-		(rev "5")
+		(title "Teapotlabs Atlas")
+		(date "2024-10-25")
+		(rev "1")
 		(company "Teapot Laboratories")
 	)
