File: hardware/kicad/main_controller.kicad_sch (KiCad schematic)
At the start: 40 parts, among them Q1 DMG1012UW, SW1 B3U-3000P, SW2 B3U-3000P, SW3 B3U-3000P, U1 ESP32-C6FH4, Y1 CM315D32768DZFT, Y2 R940000171

Commit message: update schematics info
Other:
- title: Main Controller -> Teapotlabs Atlas
Changed lines of the file:
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@@
 	(paper "A4")
 	(title_block
-		(title "Main Controller")
-		(date "2024-04-06")
-		(rev "5")
+		(title "Teapotlabs Atlas")
+		(date "2024-10-25")
+		(rev "1")
 		(company "Teapot Laboratories")
 	)
