File: hardware/kicad/power_regulator.kicad_sch (KiCad schematic)
At the start: 10 parts, among them Q8 PMV32UP, Q9 DMG1012UW, U6 XC6220

Commit message: update schematics info
Other:
- title: Power Regulator -> Teapotlabs Atlas
Changed lines of the file:
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@@
 	(paper "A4")
 	(title_block
-		(title "Power Regulator")
-		(date "2024-04-06")
-		(rev "5")
+		(title "Teapotlabs Atlas")
+		(date "2024-10-25")
+		(rev "1")
 		(company "Teapot Laboratories")
 	)
