File: hardware/kicad/sensor.kicad_sch (KiCad schematic)
At the start: 12 parts, among them Q4 PMV32UP, Q5 DMG1012UW, U7 BME688

Commit message: clean-up
Other:
- moved on the sheet: C27, C28, C29, Q4, Q5, R16, R17, R20, R21, R22, R23, U7

Commit message: update schematics info
Other:
- title: Sensor -> Teapotlabs Atlas
Changed lines of the file:
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@@
 	(paper "A4")
 	(title_block
-		(title "Sensor")
-		(date "2024-04-06")
-		(rev "5")
+		(title "Teapotlabs Atlas")
+		(date "2024-10-25")
+		(rev "1")
 		(company "Teapot Laboratories")
 	)
