File: hardware/kicad/usb_power.kicad_sch (KiCad schematic)
At the start: 15 parts, among them J1 U262-161N-4BVC11, U2 USBLC6-2P6, U3 MCP73831T-2ACI/OT

Commit message: update schematics info
Other:
- title: USB Power -> Teapotlabs Atlas
Changed lines of the file:
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@@
 	(paper "A5")
 	(title_block
-		(title "USB Power")
-		(date "2024-04-06")
-		(rev "5")
+		(title "Teapotlabs Atlas")
+		(date "2024-10-25")
+		(rev "1")
 		(company "Teapot Laboratories")
 	)
